File: Apple2Card_x44/Apple2Card.kicad_sch (KiCad schematic)
At the start: 75 parts, among them J1 ICSP, J4 Conn_01x16, J5 SERCON, J6 WIZNET 5500, SW1 SW_Push, U1 AP1117-33, U2 74HCT32, U3 74HCT00, U4 82C55A, U5 Slot1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

Commit message: x44: Updated the schematics .pdf
'Printed' the new A3 version.

Also added a Readme with a warning, as nothing has been tested yet.

Signed-off-by: Michel Pollet <buserror@gmail.com>
Other:
- company: (none) -> Daniel Marks, Michel Pollet
- title: (none) -> Apple II Arduino Interface
Changed lines of the file:
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@@
 (kicad_sch (version 20230121) (generator eeschema)
   (paper "A3")
+  (title_block
+    (title "Apple II Arduino Interface")
+    (date "2023-08-05")
+    (rev "x44_1")
+    (company "Daniel Marks, Michel Pollet")
+    (comment 1 "CC-BY-SA 4.0")
+  )
   (junction (at 298.196 185.42) (diameter 0) (color 0 0 0 0)
   )

Commit message: 644: Added a couple more LCSC properties
Somehow the slot part # hadn't been saved in the schematic. No
functional change.

Signed-off-by: Michel Pollet <buserror@gmail.com>
Parts:
- U5, U6: LCSC (none) -> C5155564
- U9: LCSC (none) -> C2874016
Changed lines of the file:
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@@
+      (effects (font (size 1.27 1.27)) hide)
+    )
+    (property "LCSC" "C2874016" (at 324.739 142.24 0)
       (effects (font (size 1.27 1.27)) hide)
     )
@@
     (property "Datasheet" "" (at 90.678 138.176 0)
       (effects (font (size 1.524 1.524)))
+    )
+    (property "LCSC" "C5155564" (at 85.598 150.876 0)
+      (effects (font (size 1.27 1.27)) hide)
     )
     (pin "2")
@@
       (effects (font (size 1.524 1.524)))
     )
-    (pin "2")
+    (property "LCSC" "C5155564" (at 85.598 183.896 0)
+      (effects (font (size 1.27 1.27)) hide)
+    )
+    (pin "2")
